File: Virulent_HW.brd (EAGLE design)
At the start: 60 parts, among them U1 STM32F050G6U6

Commit message: Updated reciever and PLL circuitry. Added hard and soft reset buttons.
Parts:
- added C27: 1n, rcl:C1206
- added C28: NU, rcl:C1206
- added D1: NTE583, Virulent_HW:NTE583
- added R22, R24: 10k, Virulent_HW:R0402
- added R23: 15k, Virulent_HW:R0402
- added R25: 6.8k, Virulent_HW:R0402
- added R26, R28: 1Meg, Virulent_HW:R0402
- added R27: 5.6Meg, Virulent_HW:R0402
- added SW1: COM08229, Virulent_HW:COM08229
- added SW2: COM08720, Virulent_HW:COM08720
- C1, C2, C3: value (none) -> 0.1u
- C13: value (none) -> 250u
- C14, C15, C16: value (none) -> 2.2u
- C17, C18, C19, C20, C21: value (none) -> 1n
- R1, R2, R3: value (none) -> 4.7k
- moved C20 291.7 mm to (-54.6, -445.8)
- moved C16 287.9 mm to (-54.6, -414.0)
- moved C13 281.7 mm to (-54.6, -396.2)
- moved C21 280.4 mm to (-54.6, -452.1)
- moved C3 279.1 mm to (-54.6, -387.4)
- moved C17 276.6 mm to (-54.6, -420.4)
- moved C2 276.6 mm to (-54.6, -378.5)
- moved C1 274.1 mm to (-54.6, -369.6)
- moved C14 259.3 mm to (-54.6, -401.3)
- moved C15 257.7 mm to (-54.6, -407.7)
- moved C18 256.8 mm to (-54.6, -426.7)
- moved C19 255.2 mm to (-54.6, -433.1)
- moved R1 252.7 mm to (-55.9, -373.4)
- moved R2 241.2 mm to (-55.9, -382.3)
- moved R3 222.4 mm to (-55.9, -391.2)
Connections:
- new net N$27: PLL3.6, R25.2
- new net N$29: D1.P$2, NFC1.1, R26.2, R27.1
- new net RESET: R22.1, SW1.2, U1.8
- net +3.3V: now also R22.2
- net +5V: now also C17.2, C18.2, C19.2, R27.2; no longer C16.1, C20.1, C3.1, PLL3.4
- net GND: now also C1.1, C13.1, C14.1, C15.1, C16.1, C17.1, C18.1, C19.1, C2.1, C20.1, C21.1, C27.1, C28.2, C3.1, R26.1, R28.1, SW1.1, SW2.3, SW2.4; no longer C1.2, C13.2, C14.2, C15.2, C16.2, C17.2, C18.2, C19.2, C2.2, C20.2, C21.2, C3.2
- net N$1: now also C1.2, PLL1.2, R1.2; no longer C1.1, PLL1.1
- net N$10: now also C15.2, PLL2.1; no longer C17.1, PLL2.5, R2.1
- net N$12: now also C21.2, PLL2.5, R24.1; no longer C18.1, PLL3.1
- net N$13: now also PLL1.6, R23.2; no longer PLL3.6, R3.2
- net N$14: now also PLL2.6, R24.2; no longer C19.1, PLL3.2
- net N$17: now also C27.2, R25.1; no longer C21.1, R3.1
- net N$2: now also C2.2, PLL2.2, R2.2; no longer C14.1, PLL2.1
- net N$3: now also C3.2, PLL3.2, R3.2; no longer PLL1.6, R1.2
- net N$4: now also C13.2, R2.1, R3.1; no longer C13.1, PLL1.5
- net N$5: now also C14.2, PLL1.1; no longer C2.1, PLL1.2
- net N$6: now also SW2.1, SW2.2
- net N$7: now also C16.2, PLL3.1; no longer PLL2.6, R2.2
- net N$8: now also C20.2, PLL1.5, R23.1; no longer C15.1, PLL2.2
- net NFC: now also C28.1, D1.P$1, R28.2; no longer NFC1.1

Commit message: updated package size for 250y Capacitor
Parts:
- added C29: NU, rcl:C1206
- added R29: 0, Virulent_HW:R0402
- C13: device rcl:C1206 -> rcl:C1210
- R28: value 1Meg -> 56k
- moved C13 124.5 mm to (-54.6, -520.7)
- moved VR1 62.7 mm to (15.2, 10.2), turned to 90 degrees
Connections:
- new net N$30: C29.1, NFC1.2, R29.1
- net +5V: now also PLL3.4
- net GND: now also C13.2; no longer C13.1
- net N$26: now also C29.2, R29.2; no longer NFC1.2
- net N$4: now also C13.1; no longer C13.2
Changed lines of the file:
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@@
 <elements>
 <element name="PLL1" library="Virulent_HW" package="SOIC-8" value="LM567CM/NOPB-ND" x="-7.62" y="-16.51"/>
-<element name="VR1" library="motorFeedback" package="PG-TO252-5-11" value="TLE4476D" x="-17.78" y="-43.18"/>
+<element name="VR1" library="motorFeedback" package="PG-TO252-5-11" value="TLE4476D" x="15.24" y="10.16" rot="R90"/>
 <element name="C4" library="rcl" package="C1206" value="0.47u" x="-19.05" y="-54.61"/>
 <element name="C5" library="rcl" package="C0402" value="0.1u" x="-20.32" y="-58.42"/>
@@
 <element name="C3" library="rcl" package="C1206" value="0.1u" x="-54.61" y="-387.35"/>
 <element name="R3" library="Virulent_HW" package="R0402" value="4.7k" x="-55.88" y="-391.16"/>
-<element name="C13" library="rcl" package="C1206" value="250u" x="-54.61" y="-396.24"/>
 <element name="C14" library="rcl" package="C1206" value="2.2u" x="-54.61" y="-401.32"/>
 <element name="C15" library="rcl" package="C1206" value="2.2u" x="-54.61" y="-407.67"/>
@@
 <element name="R27" library="Virulent_HW" package="R0402" value="5.6Meg" x="-55.88" y="-481.33"/>
 <element name="C28" library="rcl" package="C1206" value="NU" x="-54.61" y="-487.68"/>
-<element name="R28" library="Virulent_HW" package="R0402" value="1Meg" x="-55.88" y="-494.03"/>
+<element name="R28" library="Virulent_HW" package="R0402" value="56k" x="-55.88" y="-494.03"/>
 <element name="D1" library="Virulent_HW" package="NTE583" value="NTE583" x="-52.07" y="-500.38"/>
+<element name="C29" library="rcl" package="C1206" value="NU" x="-54.61" y="-508"/>
+<element name="R29" library="Virulent_HW" package="R0402" value="0" x="-55.88" y="-514.35"/>
+<element name="C13" library="rcl" package="C1210" value="250u" x="-54.61" y="-520.7"/>
 </elements>
 <signals>
@@
 <wire x1="-20.45" y1="-72.39" x2="-21.27" y2="-78.74" width="0" layer="19" extent="1-1"/>
 <wire x1="-20.97" y1="-62.23" x2="-20.45" y2="-72.39" width="0" layer="19" extent="1-1"/>
-<wire x1="-18.923" y1="-48.26" x2="-20.97" y2="-62.23" width="0" layer="19" extent="1-1"/>
+<wire x1="20.32" y1="9.017" x2="-20.97" y2="-62.23" width="0" layer="19" extent="1-1"/>
 </signal>
 <signal name="+5V">
@@
 <contactref element="C19" pad="2"/>
 <contactref element="R27" pad="2"/>
+<contactref element="PLL3" pad="4"/>
 <wire x1="-20.055" y1="-182.495" x2="-29.34" y2="-215.9" width="0" layer="19" extent="1-1"/>
-<wire x1="-15.875" y1="-140.7795" x2="-20.055" y2="-182.495" width="0" layer="19" extent="1-1"/>
+<wire x1="-15.875" y1="-168.7195" x2="-20.055" y2="-182.495" width="0" layer="19" extent="1-1"/>
+<wire x1="-15.875" y1="-140.7795" x2="-15.875" y2="-168.7195" width="0" layer="19" extent="1-1"/>
 <wire x1="-37.15" y1="-283.83" x2="-29.34" y2="-215.9" width="0" layer="19" extent="1-1"/>
 <wire x1="-20.45" y1="-67.31" x2="-15.875" y2="-140.7795" width="0" layer="19" extent="1-1"/>
 <wire x1="-20.97" y1="-58.42" x2="-20.45" y2="-67.31" width="0" layer="19" extent="1-1"/>
-<wire x1="-16.637" y1="-48.26" x2="-20.97" y2="-58.42" width="0" layer="19" extent="1-1"/>
-<wire x1="-5.715" y1="-18.8595" x2="-16.637" y2="-48.26" width="0" layer="19" extent="1-1"/>
+<wire x1="-5.715" y1="-18.8595" x2="-20.97" y2="-58.42" width="0" layer="19" extent="1-1"/>
+<wire x1="20.32" y1="11.303" x2="-5.715" y2="-18.8595" width="0" layer="19" extent="1-1"/>
 <wire x1="-53.21" y1="-420.37" x2="-37.15" y2="-283.83" width="0" layer="19" extent="1-1"/>
 <wire x1="-53.21" y1="-426.72" x2="-53.21" y2="-420.37" width="0" layer="19" extent="1-1"/>
@@
 <wire x1="-52.07" y1="-306.07" x2="-53.21" y2="-344.17" width="0" layer="19" extent="1-1"/>
 <wire x1="-20.45" y1="-54.61" x2="-52.07" y2="-306.07" width="0" layer="19" extent="1-1"/>
-<wire x1="-20.066" y1="-48.26" x2="-20.45" y2="-54.61" width="0" layer="19" extent="1-1"/>
+<wire x1="20.32" y1="7.874" x2="-20.45" y2="-54.61" width="0" layer="19" extent="1-1"/>
 </signal>
 <signal name="GND">
@@
 <contactref element="SW2" pad="3"/>
 <contactref element="SW2" pad="4"/>
-<contactref element="C13" pad="1"/>
 <contactref element="C1" pad="1"/>
 <contactref element="C2" pad="1"/>
@@
 <contactref element="C28" pad="2"/>
 <contactref element="PLL3" pad="7"/>
+<contactref element="C13" pad="2"/>
 <wire x1="-56.01" y1="-452.12" x2="-56.01" y2="-445.77" width="0" layer="19" extent="1-1"/>
 <wire x1="-56.01" y1="-433.07" x2="-56.01" y2="-445.77" width="0" layer="19" extent="1-1"/>
@@
 <wire x1="-56.01" y1="-407.67" x2="-56.01" y2="-414.02" width="0" layer="19" extent="1-1"/>
 <wire x1="-56.01" y1="-401.32" x2="-56.01" y2="-407.67" width="0" layer="19" extent="1-1"/>
-<wire x1="-56.01" y1="-396.24" x2="-56.01" y2="-401.32" width="0" layer="19" extent="1-1"/>
-<wire x1="-56.01" y1="-387.35" x2="-56.01" y2="-396.24" width="0" layer="19" extent="1-1"/>
+<wire x1="-56.01" y1="-464.82" x2="-56.01" y2="-452.12" width="0" layer="19" extent="1-1"/>
+<wire x1="-56.53" y1="-476.25" x2="-56.01" y2="-464.82" width="0" layer="19" extent="1-1"/>
+<wire x1="-53.21" y1="-487.68" x2="-56.53" y2="-476.25" width="0" layer="19" extent="1-1"/>
+<wire x1="-56.53" y1="-494.03" x2="-53.21" y2="-487.68" width="0" layer="19" extent="1-1"/>
+<wire x1="-56.01" y1="-387.35" x2="-56.01" y2="-401.32" width="0" layer="19" extent="1-1"/>
 <wire x1="-56.01" y1="-378.46" x2="-56.01" y2="-387.35" width="0" layer="19" extent="1-1"/>
 <wire x1="-56.01" y1="-369.57" x2="-56.01" y2="-378.46" width="0" layer="19" extent="1-1"/>
@@
 <wire x1="-56.27" y1="-351.79" x2="-50.24" y2="-361.37" width="0" layer="19" extent="1-1"/>
 <wire x1="-56.01" y1="-344.17" x2="-56.27" y2="-351.79" width="0" layer="19" extent="1-1"/>
-<wire x1="-56.01" y1="-464.82" x2="-56.01" y2="-452.12" width="0" layer="19" extent="1-1"/>
-<wire x1="-56.53" y1="-476.25" x2="-56.01" y2="-464.82" width="0" layer="19" extent="1-1"/>
-<wire x1="-53.21" y1="-487.68" x2="-56.53" y2="-476.25" width="0" layer="19" extent="1-1"/>
-<wire x1="-56.53" y1="-494.03" x2="-53.21" y2="-487.68" width="0" layer="19" extent="1-1"/>
+<wire x1="-53.21" y1="-520.7" x2="-56.53" y2="-494.03" width="0" layer="19" extent="1-1"/>
 <wire x1="-45.72" y1="-317.5" x2="-56.01" y2="-344.17" width="0" layer="19" extent="1-1"/>
 <wire x1="-52.07" y1="-311.15" x2="-45.72" y2="-317.5" width="0" layer="19" extent="1-1"/>
@@
 <wire x1="-19.67" y1="-58.42" x2="-19.67" y2="-62.23" width="0" layer="19" extent="1-1"/>
 <wire x1="-17.65" y1="-54.61" x2="-19.67" y2="-58.42" width="0" layer="19" extent="1-1"/>
-<wire x1="-17.78" y1="-41.6814" x2="-17.65" y2="-54.61" width="0" layer="19" extent="1-1"/>
-<wire x1="-8.255" y1="-14.1605" x2="-17.78" y2="-41.6814" width="0" layer="19" extent="1-1"/>
+<wire x1="-8.255" y1="-14.1605" x2="-17.65" y2="-54.61" width="0" layer="19" extent="1-1"/>
+<wire x1="13.7414" y1="10.16" x2="-8.255" y2="-14.1605" width="0" layer="19" extent="1-1"/>
 </signal>
 <signal name="5V_ENABLE">
 <contactref element="VR1" pad="5"/>
 <contactref element="U1" pad="7"/>
-<wire x1="-15.494" y1="-48.26" x2="-34.995" y2="-216.13" width="0" layer="19" extent="1-1"/>
+<wire x1="20.32" y1="12.446" x2="-34.995" y2="-216.13" width="0" layer="19" extent="1-1"/>
 </signal>
 <signal name="PLL_INT2">
@@
 <contactref element="CT1" pad="1"/>
 <contactref element="C25" pad="1"/>
-<contactref element="NFC1" pad="2"/>
-<wire x1="-54.61" y1="-291.83" x2="-56.01" y2="-299.72" width="0" layer="19" extent="1-1"/>
-<wire x1="-47.32" y1="-292.1" x2="-54.61" y2="-291.83" width="0" layer="19" extent="1-1"/>
+<contactref element="C29" pad="2"/>
+<contactref element="R29" pad="2"/>
+<wire x1="-47.32" y1="-292.1" x2="-56.01" y2="-299.72" width="0" layer="19" extent="1-1"/>
+<wire x1="-53.21" y1="-508" x2="-56.01" y2="-299.72" width="0" layer="19" extent="1-1"/>
+<wire x1="-55.23" y1="-514.35" x2="-53.21" y2="-508" width="0" layer="19" extent="1-1"/>
 </signal>
 <signal name="SWD_NRST">
@@
 <contactref element="R2" pad="1"/>
 <contactref element="R3" pad="1"/>
-<contactref element="C13" pad="2"/>
-<wire x1="-53.21" y1="-396.24" x2="-56.53" y2="-391.16" width="0" layer="19" extent="1-1"/>
+<contactref element="C13" pad="1"/>
 <wire x1="-56.53" y1="-382.27" x2="-56.53" y2="-391.16" width="0" layer="19" extent="1-1"/>
 <wire x1="-56.53" y1="-373.38" x2="-56.53" y2="-382.27" width="0" layer="19" extent="1-1"/>
+<wire x1="-56.01" y1="-520.7" x2="-56.53" y2="-391.16" width="0" layer="19" extent="1-1"/>
 </signal>
 <signal name="N$5">
@@
 <wire x1="-19.685" y1="-168.7195" x2="-53.21" y2="-414.02" width="0" layer="19" extent="1-1"/>
 </signal>
+<signal name="N$30">
+<contactref element="R29" pad="1"/>
+<contactref element="C29" pad="1"/>
+<contactref element="NFC1" pad="2"/>
+<wire x1="-56.01" y1="-508" x2="-54.61" y2="-291.83" width="0" layer="19" extent="1-1"/>
+<wire x1="-56.53" y1="-514.35" x2="-56.01" y2="-508" width="0" layer="19" extent="1-1"/>
+</signal>
 </signals>

Commit message: Updated uC pinout.
Connections:
- net N$11 renamed LED_GREEN
- net N$15 renamed LED_RED
- net N$16 renamed LED_BLUE
- net N$21 renamed O_GREEN
- net N$22 renamed O_RED
- net N$23 renamed O_BLUE
- net N$25 renamed TEAMID1
- net N$28 renamed TEAMID0
- removed net PLL_INT2: PLL1.8, R6.1, U1.6
- removed net PLL_INT3: PLL2.8, R7.1, U1.14
- removed net PLL_INT5: PLL3.8, R8.1, U1.2
- removed net RESET: R22.1, SW1.2, U1.8
- new net NRESET_SOFT: R22.1, SW1.2, U1.6
- new net PLL_B: PLL3.8, R8.1, U1.28
- new net PLL_G: PLL2.8, R7.1, U1.27
- new net PLL_R: PLL1.8, R6.1, U1.26
Changed lines of the file:
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@@
 <contactref element="JP1" pad="5"/>
 <contactref element="C26" pad="1"/>
-<contactref element="SW1" pad="1"/>
 <contactref element="SW2" pad="3"/>
 <contactref element="SW2" pad="4"/>
@@
 <contactref element="PLL3" pad="7"/>
 <contactref element="C13" pad="2"/>
+<contactref element="SW1" pad="1"/>
 <wire x1="-56.01" y1="-452.12" x2="-56.01" y2="-445.77" width="0" layer="19" extent="1-1"/>
 <wire x1="-56.01" y1="-433.07" x2="-56.01" y2="-445.77" width="0" layer="19" extent="1-1"/>
@@
 <wire x1="20.32" y1="12.446" x2="-34.995" y2="-216.13" width="0" layer="19" extent="1-1"/>
 </signal>
-<signal name="PLL_INT2">
-<contactref element="PLL1" pad="8"/>
-<contactref element="R6" pad="1"/>
-<contactref element="U1" pad="6"/>
-<wire x1="-33.67" y1="-222.25" x2="-34.895" y2="-215.63" width="0" layer="19" extent="1-1"/>
-<wire x1="-9.525" y1="-14.1605" x2="-34.895" y2="-215.63" width="0" layer="19" extent="1-1"/>
-</signal>
 <signal name="NFC">
 <contactref element="PLL2" pad="3"/>
@@
 <wire x1="-56.07" y1="-500.38" x2="-55.23" y2="-494.03" width="0" layer="19" extent="1-1"/>
 </signal>
-<signal name="PLL_INT3">
-<contactref element="PLL2" pad="8"/>
-<contactref element="R7" pad="1"/>
-<contactref element="U1" pad="14"/>
-<wire x1="-33.67" y1="-227.33" x2="-31.52" y2="-216.605" width="0" layer="19" extent="1-1"/>
-<wire x1="-19.685" y1="-136.0805" x2="-31.52" y2="-216.605" width="0" layer="19" extent="1-1"/>
-</signal>
-<signal name="PLL_INT5">
-<contactref element="PLL3" pad="8"/>
-<contactref element="R8" pad="1"/>
-<contactref element="U1" pad="2"/>
-<wire x1="-33.67" y1="-232.41" x2="-34.895" y2="-213.63" width="0" layer="19" extent="1-1"/>
-<wire x1="-19.685" y1="-164.0205" x2="-34.895" y2="-213.63" width="0" layer="19" extent="1-1"/>
-</signal>
 <signal name="N$18">
 <contactref element="CTX1" pad="1"/>
@@
 <wire x1="-32.37" y1="-237.49" x2="-34.995" y2="-213.13" width="0" layer="19" extent="1-1"/>
 </signal>
-<signal name="N$11">
+<signal name="LED_GREEN">
 <contactref element="RGB1" pad="1"/>
 <contactref element="R11" pad="1"/>
 <wire x1="-39.445" y1="-242.75" x2="-41.29" y2="-247.65" width="0" layer="19" extent="1-1"/>
 </signal>
-<signal name="N$15">
+<signal name="LED_RED">
 <contactref element="RGB1" pad="2"/>
 <contactref element="R12" pad="1"/>
 <wire x1="-39.045" y1="-241.7" x2="-41.29" y2="-252.73" width="0" layer="19" extent="1-1"/>
 </signal>
-<signal name="N$16">
+<signal name="LED_BLUE">
 <contactref element="RGB1" pad="3"/>
 <contactref element="R13" pad="1"/>
 <wire x1="-39.045" y1="-240.9" x2="-41.29" y2="-257.81" width="0" layer="19" extent="1-1"/>
 </signal>
-<signal name="N$21">
+<signal name="O_GREEN">
 <contactref element="R11" pad="2"/>
 <contactref element="U1" pad="15"/>
 <wire x1="-39.99" y1="-247.65" x2="-31.045" y2="-216.13" width="0" layer="19" extent="1-1"/>
 </signal>
-<signal name="N$22">
+<signal name="O_RED">
 <contactref element="R12" pad="2"/>
 <contactref element="U1" pad="24"/>
 <wire x1="-39.99" y1="-252.73" x2="-32.52" y2="-212.755" width="0" layer="19" extent="1-1"/>
 </signal>
-<signal name="N$23">
+<signal name="O_BLUE">
 <contactref element="R13" pad="2"/>
 <contactref element="U1" pad="25"/>
 <wire x1="-39.99" y1="-257.81" x2="-33.02" y2="-212.755" width="0" layer="19" extent="1-1"/>
 </signal>
-<signal name="N$25">
+<signal name="TEAMID1">
 <contactref element="U1" pad="20"/>
 <contactref element="R14" pad="1"/>
@@
 <wire x1="-39.99" y1="-267.97" x2="-41.29" y2="-262.89" width="0" layer="19" extent="1-1"/>
 </signal>
-<signal name="N$28">
+<signal name="TEAMID0">
 <contactref element="U1" pad="19"/>
 <contactref element="R16" pad="1"/>
@@
 <wire x1="-55.23" y1="-327.66" x2="-32.02" y2="-212.755" width="0" layer="19" extent="1-1"/>
 </signal>
-<signal name="RESET">
-<contactref element="U1" pad="8"/>
+<signal name="NRESET_SOFT">
 <contactref element="R22" pad="1"/>
 <contactref element="SW1" pad="2"/>
-<wire x1="-47.87" y1="-351.79" x2="-34.52" y2="-216.605" width="0" layer="19" extent="1-1"/>
+<contactref element="U1" pad="6"/>
+<wire x1="-47.87" y1="-351.79" x2="-34.895" y2="-215.63" width="0" layer="19" extent="1-1"/>
 <wire x1="-56.53" y1="-358.14" x2="-47.87" y2="-351.79" width="0" layer="19" extent="1-1"/>
 </signal>
@@
 <wire x1="-56.53" y1="-514.35" x2="-56.01" y2="-508" width="0" layer="19" extent="1-1"/>
 </signal>
+<signal name="PLL_R">
+<contactref element="PLL1" pad="8"/>
+<contactref element="R6" pad="1"/>
+<contactref element="U1" pad="26"/>
+<wire x1="-33.67" y1="-222.25" x2="-33.52" y2="-212.755" width="0" layer="19" extent="1-1"/>
+<wire x1="-9.525" y1="-14.1605" x2="-33.52" y2="-212.755" width="0" layer="19" extent="1-1"/>
+</signal>
+<signal name="PLL_B">
+<contactref element="PLL3" pad="8"/>
+<contactref element="R8" pad="1"/>
+<contactref element="U1" pad="28"/>
+<wire x1="-33.67" y1="-232.41" x2="-34.52" y2="-212.655" width="0" layer="19" extent="1-1"/>
+<wire x1="-19.685" y1="-164.0205" x2="-34.52" y2="-212.655" width="0" layer="19" extent="1-1"/>
+</signal>
+<signal name="PLL_G">
+<contactref element="PLL2" pad="8"/>
+<contactref element="R7" pad="1"/>
+<contactref element="U1" pad="27"/>
+<wire x1="-33.67" y1="-227.33" x2="-34.02" y2="-212.755" width="0" layer="19" extent="1-1"/>
+<wire x1="-19.685" y1="-136.0805" x2="-34.02" y2="-212.755" width="0" layer="19" extent="1-1"/>
+</signal>
 </signals>

Commit message: updated cap sizes. Started to mess with board layour but did not accomplish very much.
Parts:
- added C30: 0.1u, rcl:C0402
- added R31: 10k, Virulent_HW:R0402
- C1, C14, C15, C16, C17, C18, C19, C2, C20, C21, C22, C23, C24, C25, C27, C28, C29, C3: device rcl:C1206 -> rcl:C0402
- moved R29 598.5 mm to (39.5, 76.5)
- moved C29 594.0 mm to (39.5, 78.5)
- moved C13 587.8 mm to (20.6, 62.3), turned to 180 degrees
- moved D1 582.7 mm to (20.3, 77.8)
- moved R28 575.5 mm to (11.5, 77.5), turned to 90 degrees
- moved C28 569.3 mm to (13.5, 77.5), turned to 270 degrees
- moved R27 565.5 mm to (28.8, 77.8), turned to 270 degrees
- moved R26 560.1 mm to (26.5, 77.8), turned to 90 degrees
- moved R25 546.4 mm to (37.3, 67.3), turned to 180 degrees
- moved C27 538.6 mm to (37.1, 65.9)
- moved R24 527.4 mm to (37.8, 60.6), turned to 180 degrees
- moved C21 519.7 mm to (37.8, 59.3)
- moved C20 507.1 mm to (38.3, 52.8)
- moved C19 505.6 mm to (26.5, 65.9), turned to 180 degrees
- moved R23 502.5 mm to (38.3, 54.2), turned to 180 degrees
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Connections:
- removed net CARRIER_FREQ: HEX1.10, HEX1.12, HEX1.2, HEX1.4, HEX1.6, SPST1.1
- new net CHOPPED_FREQ: C24.1, HEX1.14, SPST1.2
- new net N$11: C30.2, SPST1.5
- net +5V: now also C30.1, SPST1.1; no longer C24.1, HEX1.14, SPST1.5
- net 5V_ENABLE: now also R31.2
- net GND: now also R31.1
- net NFC: now also HEX1.10, HEX1.12, HEX1.2, HEX1.4, HEX1.6; no longer SPST1.2
Routing:
- net GND: track 0.00 -> 360.0 mm
Other:
- board outline added: 100 x 80 mm

Commit message: messed around with PCB layout
Parts:
- moved CTX1 98.2 mm to (92.7, 27.1)
- moved R27 95.5 mm to (90.8, 5.12)
- moved D1 87.1 mm to (85.5, 20.0)
- moved NFC1 86.3 mm to (83.3, 7.82)
- moved R26 83.9 mm to (82.0, 14.9)
- moved C24 82.9 mm to (82.7, 27.4)
- moved C29 80.8 mm to (90.3, 15.7)
- moved C25 80.1 mm to (89.5, 9.46)
- moved CT1 80.1 mm to (89.4, 12.0)
- moved R29 80.1 mm to (84.9, 10.5)
- moved HEX1 78.7 mm to (85.5, 38.5)
- moved C30 76.3 mm to (76.4, 23.4)
- moved JP1 69.0 mm to (59.0, 9.84)
- moved R4 64.8 mm to (15.2, 14.1)
- moved R5 64.8 mm to (18.2, 14.2)
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Routing:
- net STM_SWDAT: track 0.00 -> 27.5 mm, vias 0 -> 2
- net STM_SWCLK: track 0.00 -> 25.6 mm, vias 0 -> 2
- net +3.3V: track 0.00 -> 24.5 mm, vias 0 -> 4
- net STM_SWO: track 0.00 -> 24.4 mm, vias 0 -> 2
- net +5V: track 0.00 -> 23.4 mm, vias 0 -> 2
- net PLL_R: track 0.00 -> 23.0 mm
- net NFC: track 0.00 -> 22.1 mm, vias 0 -> 3
- net N$4: track 0.00 -> 22.0 mm, vias 0 -> 3
- net PLL_B: track 0.00 -> 21.1 mm
- net N$6: track 0.00 -> 19.8 mm, vias 0 -> 2
- net PLL_G: track 0.00 -> 16.5 mm
- net N$2: track 0.00 -> 9.66 mm
- net N$1: track 0.00 -> 9.10 mm
- net N$3: track 0.00 -> 8.96 mm
- net N$8: track 0.00 -> 5.75 mm
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